File: raven-split-38key/raven-split-38key__choc-hotswap-n!n/pcb/raven-split-38key__choc-hotswap-n!n.kicad_pcb (KiCad board)
At the start: 2 copper layers, 124.4 x 86 mm, 45 parts, among them M2_0 MountingHole_2.2mm_M2_Pad, M2_1 MountingHole_2.2mm_M2_Pad, SW10 SW_PUSH, SW11 SW_PUSH, SW12 SW_PUSH, SW14 SW_PUSH, SW15 SW_PUSH, SW16 SW_PUSH, SW17 SW_PUSH, SW18 SW_PUSH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

Commit message: generate gerbers, update README and test
Parts:
- added G***: LOGO, LOGO, F.Cu at (152.3, 73.9)
- added G***: LOGO, LOGO, B.Cu at (152.4, 74.0)
- added SW_POWER: SW_SPDT, Kailh:SPDT_C128955, F.Cu at (153.4, 57.4)
- SW_POWER: moved to B.Cu
- turned SW_POWER to 180 degrees
Routing:
- net col3: track 0.00 -> 216.2 mm, vias 0 -> 4
- net col1: track 0.00 -> 196.4 mm, vias 0 -> 3
- net col2: track 0.00 -> 192.6 mm, vias 0 -> 3
- net row1: track 0.00 -> 192.6 mm, vias 0 -> 6
- net col4: track 0.00 -> 189.2 mm, vias 0 -> 4
- net row2: track 0.00 -> 185.2 mm, vias 0 -> 5
- net col5: track 0.00 -> 180.2 mm, vias 0 -> 4
- net col0: track 0.00 -> 152.4 mm, vias 0 -> 1
- net row0: track 0.00 -> 148.9 mm, vias 0 -> 5
- net row3: track 0.00 -> 103.6 mm, vias 0 -> 3
- net GND: track 0.00 -> 62.6 mm
- net reset: track 0.00 -> 56.3 mm
- net Net-(U1-Pad24): track 0.00 -> 25.4 mm
- net Net-(D21-Pad2): track 0.00 -> 23.0 mm, vias 0 -> 1
- net Net-(D12-Pad2): track 0.00 -> 22.7 mm, vias 0 -> 1
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